Commit message: Complete Q1(c): substitute collision meshes with box geometries in URDF

File: armando_description/urdf/arm.urdf (robot description, URDF)
Before this commit: robot arm, 17 links, 16 joints
Links:
- link base_link: geometry collision box size=0.10 0.10 0.035; visual mesh filename=package://armando_description/meshes/base_link.stl scale=0.001 0.001 0.001
- link base_turn: geometry collision box size=0.08 0.08 0.05; visual mesh filename=package://armando_description/meshes/base_turn.stl scale=0.001 0.001 0.001
- link base_turn_rot: geometry collision box size=0.08 0.08 0.04; visual mesh filename=package://armando_description/meshes/base_turn_table_rot.stl scale=0.001 0.001 0.001
- link crawer_base: geometry collision box size=0.05 0.035 0.025; visual mesh filename=package://armando_description/meshes/the_crawer_base.stl scale=0.001 0.001 0.001
- link crawer_left: geometry collision box size=0.025 0.10 0.015; visual mesh filename=package://armando_description/meshes/the_crawer.stl scale=0.001 0.001 0.001
- link crawer_right: geometry collision box size=0.025 0.10 0.015; visual mesh filename=package://armando_description/meshes/the_crawer.stl scale=0.001 0.001 0.001
- link dyn2: geometry collision box size=0.09 0.04 0.010; visual mesh filename=package://armando_description/meshes/dyn.stl scale=0.01 0.01 0.01
- link dyn3: geometry collision box size=0.12 0.06 0.06; visual mesh filename=package://armando_description/meshes/dyn.stl scale=0.01 0.01 0.01
- link dyn4: geometry collision box size=0.03 0.03 0.06; visual mesh filename=package://armando_description/meshes/dyn.stl scale=0.01 0.01 0.01
- link dyn5: geometry collision box size=0.03 0.03 0.06; visual mesh filename=package://armando_description/meshes/dyn.stl scale=0.01 0.01 0.01
- link f4: geometry collision box size=0.06 0.025 0.025; visual mesh filename=package://armando_description/meshes/f4_n_f3.stl scale=0.001 0.001 0.001
- link f5: geometry collision box size=0.06 0.025 0.025; visual mesh filename=package://armando_description/meshes/f4_n_f3.stl scale=0.001 0.001 0.001
- link wrist: geometry collision box size=0.04 0.03 0.03; visual mesh filename=package://armando_description/meshes/wrist.stl scale=0.001 0.001 0.001
