Commit message: Complete Q2(c): Gazebo ros2_control controllers

File: armando_description/urdf/arm.urdf.xacro (robot description, xacro)
@@ -349,3 +349,15 @@
   </link>
 <xacro:armando_hardware_interface/>
+<gazebo>
+    <plugin
+        filename="gz_ros2_control-system"
+        name="gz_ros2_control::GazeboSimROS2ControlPlugin">
+       <parameters>
+           $(find armando_description)/config/armando_controllers.yaml
+       </parameters>
+       <controller_manager_prefix_node_name>
+           controller_manager
+       </controller_manager_prefix_node_name>
+   </plugin>
+</gazebo>
 </robot>

File: armando_description/urdf/armando_hardware_interface.xacro (robot description, xacro)
@@ -1,62 +1,26 @@
 <?xml version="1.0"?>
 <robot xmlns:xacro="http://www.ros.org/wiki/xacro">
-    <!--
-        Armando ROS2 Control Hardware Interface
-        Defines the connection between:
-        ROS2 controllers
-              |
-        ros2_control
-              |
-        Ignition Gazebo
-              |
-        Armando joints
-    -->
-    <xacro:macro name="armando_hardware_interface">
-        <ros2_control
-            name="ArmandoHardwareInterface"
-            type="system">
-            <hardware>
-                <!-- Gazebo Ignition ROS2 control plugin -->
-                <plugin>
-                    ign_ros2_control/IgnitionSystem
-                </plugin>
-            </hardware>
-            <!-- Joint 0 -->
-            <joint name="j0">
-                <command_interface name="position">
-                </command_interface>
-                <state_interface name="position">
-                </state_interface>
-                <state_interface name="velocity">
-                </state_interface>
-            </joint>
-            <!-- Joint 1 -->
-            <joint name="j1">
-                <command_interface name="position">
-                </command_interface>
-                <state_interface name="position">
-                </state_interface>
-                <state_interface name="velocity">
-                </state_interface>
-            </joint>
-            <!-- Joint 2 -->
-            <joint name="j2">
-                <command_interface name="position">
-                </command_interface>
-                <state_interface name="position">
-                </state_interface>
-                <state_interface name="velocity">
-                </state_interface>
-            </joint>
-            <!-- Joint 3 -->
-            <joint name="j3">
-                <command_interface name="position">
-                </command_interface>
-                <state_interface name="position">
-                </state_interface>
-                <state_interface name="velocity">
-                </state_interface>
-            </joint>
-        </ros2_control>
-    </xacro:macro>
+  <xacro:macro name="armando_hardware_interface">
+    <ros2_control name="HardwareInterface_Gazebo" type="system">
+      <hardware>
+        <plugin>gz_ros2_control/GazeboSimSystem</plugin>
+      </hardware>
+      <joint name="j0">
+        <command_interface name="position"/>
+        <state_interface name="position"/>
+      </joint>
+      <joint name="j1">
+        <command_interface name="position"/>
+        <state_interface name="position"/>
+      </joint>
+      <joint name="j2">
+        <command_interface name="position"/>
+        <state_interface name="position"/>
+      </joint>
+      <joint name="j3">
+        <command_interface name="position"/>
+        <state_interface name="position"/>
+      </joint>
+    </ros2_control>
+  </xacro:macro>
 </robot>

Commit message: Q3_a:Add camera link and fixed camera joint for Q3a

File: armando_description/urdf/arm.urdf.xacro (robot description, xacro)
@@ -28,4 +28,32 @@
     <child link="base_turn"/>
     <origin xyz="-0.0011 -0.011 0.05"/>
+  </joint>
+  <!-- : Camera link -->
+  <link name="camera_link">
+    <visual>
+      <geometry>
+        <box size="0.05 0.05 0.05"/>
+      </geometry>
+    </visual>
+    <collision>
+      <geometry>
+        <box size="0.05 0.05 0.05"/>
+      </geometry>
+    </collision>
+    <inertial>
+      <mass value="0.01"/>
+      <inertia
+        ixx="0.00001"
+        ixy="0.0"
+        ixz="0.0"
+        iyy="0.00001"
+        iyz="0.0"
+        izz="0.00001"/>
+    </inertial>
+  </link>
+  <joint name="camera_joint" type="fixed">
+    <parent link="base_link"/>
+    <child link="camera_link"/>
+     <origin xyz="0.04 0 0.045" rpy="0 0 0"/>
   </joint>
   <link name="base_turn">
